Commit message: update

File: ros_master/ros_package/bumperbot_description/urdf/bumperbot_description.urdf.xacro (robot description, xacro)
@@ -1,13 +1,16 @@
 <?xml version="1.0"?>
 <robot name="bumperbot" xmlns:xacro="http://ros.org/wiki/xacro">
+    <!-- Include other xacro files -->
     <xacro:include filename="$(find bumperbot_description)/urdf/bumperbot_gazebo.xacro"/>
+    <!-- Base footprint link -->
     <link name="base_footprint"/>
+    <!-- Base link -->
     <link name="base_link">
         <inertial>
             <origin xyz="0 0 0.04" rpy="0.0 0.25 0.3" />
-            <mass value="8.2573504e-01"/>
-            <inertia ixx="2.2124416e-02" ixy="-1.2294101e-04" ixz="3.4938785e-04"
-                     iyy="2.1193702e-02" iyz="-5.0120904e-05"
-                     izz="2.0064271e-02" />
+            <mass value="0.82573504"/>
+            <inertia ixx="0.022124416" ixy="-0.000122941" ixz="0.00034938785"
+                     iyy="0.021193702" iyz="-0.000050120904"
+                     izz="0.020064271" />
         </inertial>
         <visual>
@@ -17,11 +20,12 @@
             </geometry>
         </visual>
-        <collison>
+        <collision>
             <origin rpy="0 0 0" xyz="0 0 0"/>
             <geometry>
                 <mesh filename="package://bumperbot_description/meshes/base_link.STL"/>
             </geometry>
-        </collison>
+        </collision>
     </link>
+    <!-- Base joint -->
     <joint name="base_joint" type="fixed">
         <parent link="base_footprint"/>
@@ -29,11 +33,12 @@
         <origin rpy="0 0 0" xyz="0 0 0.033"/>
     </joint>
+    <!-- Right wheel link -->
     <link name="wheel_right_link">
         <inertial>
             <origin xyz="0 -0.014 0" rpy="0 0 0" />
-            <mass value="0.0530086090966721" />
-            <inertia ixx="1.88176298336665E-05" ixy="-4.8444933029987E-10" ixz="1.88163708851143E-08"
-                     iyy="3.11510738647764E-05" iyz="-6.93560663069607E-11"
-                     izz="1.8801969558182E-05" />
+            <mass value="0.0530086" />
+            <inertia ixx="1.881763e-05" ixy="-4.8444933e-10" ixz="1.8816371e-08"
+                     iyy="3.1151074e-05" iyz="-6.9356066e-11"
+                     izz="1.880197e-05" />
         </inertial>
         <visual>
@@ -43,11 +48,12 @@
             </geometry>
         </visual>
-        <collison>
+        <collision>
             <origin rpy="0 -0.015 0" xyz="0 0 0"/>
             <geometry>
                 <sphere radius="0.033"/>
             </geometry>
-        </collison>
+        </collision>
     </link>
+    <!-- Right wheel joint -->
     <joint name="wheel_right_joint" type="continuous">
         <parent link="base_link"/>
@@ -56,11 +62,12 @@
         <origin rpy="0 0 0" xyz="0 -0.07 0"/>
     </joint>
+    <!-- Left wheel link -->
     <link name="wheel_left_link">
         <inertial>
             <origin xyz="0 0.014 0" rpy="0 0 0" />
-            <mass value="0.0530086043217644" />
-            <inertia ixx="1.8792911368909E-05"  ixy="3.31256392204584E-10" ixz="-1.14082001662767E-08"
-                     iyy="3.11510738759073E-05" iyz="-3.60499245082192E-10"
-                     izz="1.88266886146847E-05" />
+            <mass value="0.0530086" />
+            <inertia ixx="1.8792911e-05" ixy="3.3125639e-10" ixz="-1.140820e-08"
+                     iyy="3.1151074e-05" iyz="-3.6049925e-10"
+                     izz="1.8826689e-05" />
         </inertial>
         <visual>
@@ -70,11 +77,12 @@
             <origin rpy="-1.57 0 0" xyz="0 0 0"/>
         </visual>
-        <collison>
+        <collision>
             <origin rpy="0 0.015 0" xyz="0 0 0"/>
             <geometry>
-                <sphere radius="0.033">
+                <sphere radius="0.033"/>
             </geometry>
-        </collison>
+        </collision>
     </link>
+    <!-- Left wheel joint -->
     <joint name="wheel_left_joint" type="continuous">
         <parent link="base_link"/>
@@ -83,11 +91,12 @@
         <origin rpy="0 0 0" xyz="0 0.07 0"/>
     </joint>
+    <!-- Front caster link -->
     <link name="caster_front_link">
         <inertial>
-            <origin xyz="3.89968128948481E-07 2.40073004698083E-07 0.00219173397061506" rpy="0 0 0" />
-            <mass value="1.44379265037903E-06" />
-            <inertia ixx="7.23075276010246E-11" ixy="-6.10956883467859E-16" ixz="2.22849693525031E-15"
-                     iyy="3.8713793085917E-11"  iyz="2.93909858781952E-15"
-                     izz="1.00967486676306E-10" />
+            <origin xyz="3.8996813e-07 2.4007300e-07 0.00219173397061506" rpy="0 0 0" />
+            <mass value="1.4437927e-06" />
+            <inertia ixx="7.2307528e-11" ixy="-6.1095688e-16" ixz="2.2284969e-15"
+                     iyy="3.8713793e-11" iyz="2.9390986e-15"
+                     izz="1.0096749e-10" />
         </inertial>
         <visual>
@@ -97,11 +106,12 @@
             <origin rpy="0 0 0" xyz="0 0 0"/>
         </visual>
-        <collison>
+        <collision>
             <origin xyz="0 0 0" rpy="0 0 0"/>
             <geometry>
                 <sphere radius="0.005"/>
             </geometry>
-        </collison>
+        </collision>
     </link>
+    <!-- Front caster joint -->
     <joint name="caster_front_joint" type="fixed">
         <parent link="base_link"/>
@@ -109,11 +119,12 @@
         <origin rpy="0 0 0" xyz="0.0475 0 -0.0275"/>
     </joint>
+    <!-- Rear caster link -->
     <link name="caster_rear_link">
         <inertial>
-            <origin xyz="3.8996812895542E-07 2.40073004698083E-07 0.00219173397061509" rpy="0 0 0" />
-            <mass value="1.44379265037902E-06" />
-            <inertia ixx="7.23075276010246E-11" ixy="-6.10956872363424E-16" ixz="2.22849693527207E-15"
-                     iyy="3.87137930859167E-11" iyz="2.939098587861E-15"
-                     izz="1.00967486676306E-10" />
+            <origin xyz="3.8996813e-07 2.4007300e-07 0.00219173397061509" rpy="0 0 0" />
+            <mass value="1.4437927e-06" />
+            <inertia ixx="7.2307528e-11" ixy="-6.1095687e-16" ixz="2.2284969e-15"
+                     iyy="3.8713793e-11" iyz="2.9390986e-15"
+                     izz="1.0096749e-10" />
         </inertial>
         <visual>
@@ -123,11 +134,12 @@
             <origin rpy="0 0 0" xyz="0 0 0"/>
         </visual>
-        <collison>
+        <collision>
             <origin xyz="0 0 0" rpy="0 0 0"/>
             <geometry>
                 <sphere radius="0.005"/>
             </geometry>
-        </collison>
+        </collision>
     </link>
+    <!-- Rear caster joint -->
     <joint name="caster_rear_joint" type="fixed">
         <parent link="base_link"/>
@@ -135,5 +147,6 @@
         <origin rpy="0 0 0" xyz="-0.0475 0 -0.0275"/>
     </joint>
-    <!-- <link name="can_link">
+    <!-- Example for an additional link (commented out)
+    <link name="can_link">
         <visual>
             <geometry>
@@ -142,9 +155,10 @@
             <origin rpy="0 0 0" xyz="0 0 0"/>
         </visual>
-    </link> -->
-    <!-- <joint name="can_joint" type="fixed">
+    </link>
+    <joint name="can_joint" type="fixed">
         <parent link="base_link"/>
         <child link="can_link"/>
         <origin rpy="1.57 0 0" xyz="-0.03 0.03 0.078"/>
-    </joint> -->
+    </joint>
+    -->
 </robot>

File: ros_master/ros_package/bumperbot_description/urdf/bumperbot_gazebo.xacro (robot description, xacro)
@@ -1,42 +1,42 @@
 <?xml version="1.0"?>
 <robot name="bumperbot" xmlns:xacro="http://ros.org/wiki/xacro">
+    <!-- Right wheel gazebo parameters -->
     <gazebo reference="wheel_right_link">
-        <mu1>100000000000000.0</mu1>
-        <mu2>100000000000000.0</mu2>
-        <kp>1000000000000.0</kp>
+        <mu1>1e14</mu1> <!-- Friction coefficient -->
+        <mu2>1e14</mu2> <!-- Friction coefficient -->
+        <kp>1e12</kp>   <!-- Spring coefficient -->
+        <kd>10</kd>     <!-- Damping coefficient -->
+        <minDepth>0.001</minDepth> <!-- Minimum penetration depth -->
+        <maxVel>0.1</maxVel>       <!-- Maximum velocity -->
+        <fdir1>1 0 0</fdir1>       <!-- Rotation direction X -->
+    </gazebo>
+    <!-- Left wheel gazebo parameters -->
+    <gazebo reference="wheel_left_link">
+        <mu1>1e14</mu1>
+        <mu2>1e14</mu2>
+        <kp>1e12</kp>
         <kd>10</kd>
         <minDepth>0.001</minDepth>
         <maxVel>0.1</maxVel>
-        <!-- rotation direction X -->
         <fdir1>1 0 0</fdir1>
     </gazebo>
-    <gazebo reference="wheel_left_link">
-        <mu1>100000000000000.0</mu1>
-        <mu2>100000000000000.0</mu2>
-        <kp>1000000000000.0</kp>
-        <kd>10</kd>
-        <minDepth>0.001</minDepth>
-        <maxVel>0.1</maxVel>
-        <!-- rotation direction X -->
-        <fdir1>1 0 0</fdir1>
-    </gazebo>
+    <!-- Front caster wheel gazebo parameters -->
     <gazebo reference="caster_front_link">
         <mu1>0.1</mu1>
         <mu2>0.1</mu2>
-        <kp>1000000.0</kp>
+        <kp>1e6</kp>
         <kd>100</kd>
         <minDepth>0.001</minDepth>
         <maxVel>0.1</maxVel>
-        <!-- rotation direction X -->
         <fdir1>1 0 0</fdir1>
     </gazebo>
-        <gazebo reference="caster_rear_link">
+    <!-- Rear caster wheel gazebo parameters -->
+    <gazebo reference="caster_rear_link">
         <mu1>0.1</mu1>
         <mu2>0.1</mu2>
-        <kp>1000000.0</kp>
+        <kp>1e6</kp>
         <kd>100</kd>
         <minDepth>0.001</minDepth>
         <maxVel>0.1</maxVel>
-        <!-- rotation direction X -->
         <fdir1>1 0 0</fdir1>
     </gazebo>
